File: Camera_Module_PCB/Power Supply.kicad_sch (KiCad schematic)
At the start: 27 parts, among them J1 SS-52400-002, SW1 SW_DIP_x01

Commit message: Made Minor Changes and Reviewed Schematic
Only a few more connections must be made to the ESP32 component. All other components should be complete.
Connections:
- net +3.3VA: no longer names the net of 3V3_R.2 (OUTPUT), C3.1, L1.1
Changed lines of the file:
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@@
 	)
 	(junction
-		(at 171.45 139.7)
-		(diameter 0)
-		(color 0 0 0 0)
-	)
-	(junction
 		(at 265.43 41.91)
 		(diameter 0)
@@
 	(wire
 		(pts
-			(xy 171.45 139.7) (xy 171.45 148.59)
-		)
-		(stroke
-			(width 0)
-			(type default)
-		)
-	)
-	(wire
-		(pts
 			(xy 30.48 45.72) (xy 30.48 46.99)
 		)
@@
 	(wire
 		(pts
-			(xy 171.45 139.7) (xy 177.8 139.7)
-		)
-		(stroke
-			(width 0)
-			(type default)
-		)
-	)
-	(wire
-		(pts
 			(xy 252.73 66.04) (xy 260.35 66.04)
 		)
@@
 	(wire
 		(pts
-			(xy 162.56 139.7) (xy 171.45 139.7)
-		)
-		(stroke
-			(width 0)
-			(type default)
-		)
-	)
-	(wire
-		(pts
-			(xy 171.45 148.59) (xy 172.72 148.59)
+			(xy 162.56 139.7) (xy 177.8 139.7)
 		)
 		(stroke
@@
 					(unit 1)
 				)
-			)
-		)
-	)
-	(symbol
-		(lib_id "power:+3.3VA")
-		(at 172.72 148.59 270)
-		(unit 1)
-		(exclude_from_sim no)
-		(in_bom yes)
-		(on_board yes)
-		(dnp no)
-		(fields_autoplaced yes)
-		(property "Reference" "#PWR0115"
-			(at 168.91 148.59 0)
-			(effects
-				(font
-					(size 1.27 1.27)
-				)
-				(hide yes)
-			)
-		)
-		(property "Value" "+3.3VA"
-			(at 176.53 148.5899 90)
-			(effects
-				(font
-					(size 1.27 1.27)
-				)
-				(justify left)
-			)
-		)
-		(property "Footprint" ""
-			(at 172.72 148.59 0)
-			(effects
-				(font
-					(size 1.27 1.27)
-				)
-				(hide yes)
-			)
-		)
-		(property "Datasheet" ""
-			(at 172.72 148.59 0)
-			(effects
-				(font
-					(size 1.27 1.27)
-				)
-				(hide yes)
-			)
-		)
-		(property "Description" "Power symbol creates a global label with name \"+3.3VA\""
-			(at 172.72 148.59 0)
-			(effects
-				(font
-					(size 1.27 1.27)
-				)
-				(hide yes)
-			)
-		)
-		(pin "1"
-		)
-		(instances
-			(project ""
-				(path "/e3d5a9d6-7dc8-43b3-bd64-189ae9cbab33/097e721d-c536-4567-9b5e-193861a3bee4"
-					(reference "#PWR0115")
-					(unit 1)
-				)
